Commit message: Addressed comments to add teleop.launch and messed around with odom (found that slowing the robot was what actually improved results the most)

File: catkin_mapmyworld/src/map_my_world/urdf/my_robot.xacro (robot description, xacro)
@@ -62,5 +62,5 @@
     <axis xyz="0 1 0" rpy="0 0 0"/>
     <limit effort="10000" velocity="1000"/>
-    <dynamics damping="1.0" friction="1.0"/>
+    <dynamics damping="0.0" friction="0.0"/>
   </joint>
   <link name='left_wheel'>
@@ -94,5 +94,5 @@
     <axis xyz="0 1 0" rpy="0 0 0"/>
     <limit effort="10000" velocity="1000"/>
-    <dynamics damping="1.0" friction="1.0"/>
+    <dynamics damping="0.0" friction="0.0"/>
   </joint>
   <link name='right_wheel'>
